File: forkboard-pcb/forkboard-pcb.kicad_sch (KiCad schematic)
At the start: 108 parts, among them J1 USB_B_Micro, J2 Conn_01x02, J3 Conn_02x18_Odd_Even, J4 Conn_02x18_Odd_Even, U1 NCP1117-3.3_SOT223, U2 W25Q128JVS, U3 RP2040, Y1 ABLS-12.000MHZ-B4-T

Commit message: added LEDS, encoder and second micro, still need to relable board 2 nets
Parts:
- removed C17: 10u, Capacitor_SMD:C_0805_2012Metric, symbol Device:C
- removed J3, J4: Conn_02x18_Odd_Even, Connector_PinHeader_2.54mm:PinHeader_2x18_P2.54mm_Vertical, symbol Connector_Generic:Conn_02x18_Odd_Even
- added C18, C19: 10nF, Capacitor_SMD:C_0402_1005Metric, symbol Device:C
- added C20: 1uF, Capacitor_SMD:C_0402_1005Metric, symbol Device:C
- added C21, C22: 27p, Capacitor_SMD:C_0402_1005Metric, symbol Device:C
- added C23, C27: 10u, Capacitor_SMD:C_0805_2012Metric, symbol Device:C
- added C24, C25, C28, C30, C31, C32, C33, C34, C35, C36: 100n, Capacitor_SMD:C_0402_1005Metric, symbol Device:C
- added C26, C29: 1u, Capacitor_SMD:C_0402_1005Metric, symbol Device:C
- added D38, D39, D40, D41, D42: LED, symbol Device:LED
- added D43, D44, D45, D46: ESD5Zxx, Diode_SMD:D_SOD-523, symbol Diode:ESD5Zxx
- added J5, J8: Conn_01x04, symbol Connector_Generic:Conn_01x04
- added J6: USB_B_Micro, RP2040_minimal:USB_Micro-B_Amphenol_10103594-0001LF_Horizontal_modified, symbol RP2040_minimal-rescue:USB_B_Micro-Connector
- added J7: Conn_01x02, Connector_PinHeader_2.54mm:PinHeader_1x02_P2.54mm_Vertical, symbol Connector_Generic:Conn_01x02
- added R10, R11, R8, R9: 10k, Capacitor_SMD:C_0402_1005Metric, symbol Device:R
- added R12, R13, R14, R15, R16: 499, Capacitor_SMD:C_0402_1005Metric, symbol Device:R
- added R17, R18: 1k, Capacitor_SMD:C_0402_1005Metric, symbol Device:R
- added R19: DNF, Capacitor_SMD:C_0402_1005Metric, symbol Device:R
- added R20, R21: 27, Capacitor_SMD:C_0402_1005Metric, symbol Device:R
- added R22, R23, R6, R7: 0, Capacitor_SMD:C_0402_1005Metric, symbol Device:R
- added SW2: RotaryEncoder, symbol Device:RotaryEncoder
- added U4: NCP1117-3.3_SOT223, Package_TO_SOT_SMD:SOT-223-3_TabPin2, symbol Regulator_Linear:NCP1117-3.3_SOT223
- added U5: RP2040, RP2040_minimal:RP2040-QFN-56, symbol MCU_RaspberryPi_RP2040:RP2040
- added U6: W25Q128JVS, Package_SO:SOIC-8_5.23x5.23mm_P1.27mm, symbol RP2040_minimal-rescue:W25Q128JVS-Memory_Flash
- added Y2: ABLS-12.000MHZ-B4-T, RP2040_minimal:Crystal_SMD_HC49-US, symbol Device:Crystal
Connections:
- net GPIO13 is gone; now on net ROW0: U3.16 (GPIO13)
- net GPIO14 is gone; now on net ROW1: U3.17 (GPIO14)
- net GPIO15 is gone; now on net ROW2: U3.18 (GPIO15)
- net GPIO16 is gone; now on net ROW3: U3.27 (GPIO16)
- net GPIO17 is gone; now on net ROW4: U3.28 (GPIO17)
- net GPIO18 is gone; now on net ROW5: U3.29 (GPIO18)
- net GPIO19 is gone; now on net COL0: U3.30 (GPIO19)
- net GPIO20 is gone; now on net COL1: U3.31 (GPIO20)
- net GPIO21 is gone; now on net COL2: U3.32 (GPIO21)
- net GPIO22 is gone; now on net COL3: U3.34 (GPIO22)
- net GPIO23 is gone; now on net COL4: U3.35 (GPIO23)
- net GPIO24 is gone; now on net COL5: U3.36 (GPIO24)
- net GPIO25 is gone; now on net COL6: U3.37 (GPIO25)
- net +1V1: now also C24.1, C25.1, C26.1, U5.23 (DVDD), U5.45 (VREG_VOUT), U5.50 (DVDD)
- net +3V3: now also C20.1, C27.1, C28.1, C29.1, C30.1, C31.1, C32.1, C33.1, C34.1, C35.1, C36.1, D38.2 (A), D39.2 (A), D40.2 (A), D41.2 (A), D42.2 (A), R10.1, R19.1, R9.2, U4.2 (VO), U5.1 (IOVDD), U5.10 (IOVDD), U5.22 (IOVDD), U5.33 (IOVDD), U5.42 (IOVDD), U5.43 (ADC_AVDD), U5.44 (VREG_IN), U5.48 (USB_VDD), U5.49 (IOVDD), U6.8 (VCC)
- net GND: now also C18.2, C19.2, C20.2, C21.2, C22.2, C23.2, C24.2, C25.2, C26.2, C27.2, C28.2, C29.2, C30.2, C31.2, C32.2, C33.2, C34.2, C35.2, C36.2, D43.2 (A), D44.2 (A), D45.2 (A), D46.2 (A), J5.4 (Pin_4), J6.5 (GND), J6.6 (Shield), J7.2 (Pin_2), J8.4 (Pin_4), SW2.C, U4.1 (GND), U5.19 (TESTEN), U5.57 (GND), U6.4 (GND)
- net GPIO2: now also U5.4 (GPIO2)
- net GPIO26_ADC0: now also U5.38 (GPIO26_ADC0)
- net GPIO27_ADC1: now also U5.39 (GPIO27_ADC1)
- net GPIO28_ADC2: now also U5.40 (GPIO28_ADC2)
- net GPIO29_ADC3: now also U5.41 (GPIO29_ADC3)
- net GPIO3: now also U5.5 (GPIO3)
- net GPIO6: now also U5.8 (GPIO6)
- net GPIO7: now also U5.9 (GPIO7)
- net QSPI_SCLK: now also U5.52 (QSPI_SCLK), U6.6 (CLK)
- net QSPI_SD0: now also U5.53 (QSPI_SD0), U6.5 (DI(IO0))
- net QSPI_SD1: now also U5.55 (QSPI_SD1), U6.2 (DO(IO1))
- net QSPI_SD2: now also U5.54 (QSPI_SD2), U6.3 (IO2)
- net QSPI_SD3: now also U5.51 (QSPI_SD3), U6.7 (IO3)
- net QSPI_SS: now also R18.1, R19.2, U5.56 (QSPI_SS), U6.1 (~{CS})
- net RUN: now also U5.26 (RUN)
- net SWCLK: now also U5.24 (SWCLK)
- net SWD: now also U5.25 (SWD)
- net USB_D+: now also J6.3 (D+), R20.1
- net USB_D-: now also J6.2 (D-), R21.1
- net VBUS: now also C23.1, J5.1 (Pin_1), J6.1 (VBUS), J8.1 (Pin_1), U4.3 (VI)
- net XIN: now also C21.1, U5.20 (XIN), Y2.1
- net XOUT: now also R17.1, U5.21 (XOUT)
- net ~{USB_BOOT}: now also J7.1 (Pin_1), R18.2
- net GPIO0: no longer names the net of U3.2 (GPIO0)
- net GPIO1: no longer names the net of U3.3 (GPIO1)
- net GPIO10: no longer names the net of U3.13 (GPIO10)
- net GPIO11: no longer names the net of U3.14 (GPIO11)
- net GPIO12: no longer names the net of U3.15 (GPIO12)
- net GPIO4 renamed UART1_TX
- net UART1_TX: now also R6.2
- net GPIO5 renamed UART1_RX
- net UART1_RX: now also R7.2
- net GPIO8: no longer names the net of U3.11 (GPIO8)
- net GPIO9: no longer names the net of U3.12 (GPIO9)
- new net: C22.1, R17.2, Y2.2
- new net: D42.1 (K), R16.2
- new net: D38.1 (K), R12.2
- new net: D40.1 (K), R14.2
- new net: R8.1, R9.1, SW2.A
- new net: D43.1 (K), J5.2 (Pin_2), R6.1
- new net: D39.1 (K), R13.2
- new net: D44.1 (K), J5.3 (Pin_3), R7.1
- new net: D46.1 (K), J8.3 (Pin_3), R23.1
- new net: R10.2, R11.2, SW2.B
- new net: R21.2, U5.46 (USB_DM)
- new net: R20.2, U5.47 (USB_DP)
- new net: D41.1 (K), R15.2
- new net: D45.1 (K), J8.2 (Pin_2), R22.1
- new net EN_SIG_A: C18.1, R8.2, U5.3 (GPIO1)
- new net EN_SIG_B: C19.1, R11.1, U5.2 (GPIO0)
- new net LED1: R16.1, U5.11 (GPIO8)
- new net LED2: R15.1, U5.12 (GPIO9)
- new net LED3: R14.1, U5.13 (GPIO10)
- new net LED4: R13.1, U5.14 (GPIO11)
- new net LED5: R12.1, U5.15 (GPIO12)
- new net UART1_RX_B2: R23.2, U5.7 (GPIO5)
- new net UART1_TX_B2: R22.2, U5.6 (GPIO4)
- no-connect marks 1 -> 2
Other:
- note removed: "IOs"

Commit message: updated board 2 net labels, still needs board 2 matrix added and usb ESD diodes
Connections:
- net +3V3: no longer C20.1, C27.1, C33.1, D38.2 (A), D39.2 (A), D40.2 (A), D41.2 (A), D42.2 (A), R19.1, U4.2 (VO), U6.8 (VCC)
- net GPIO2: no longer U5.4 (GPIO2)
- net GPIO26_ADC0: no longer U5.38 (GPIO26_ADC0)
- net GPIO27_ADC1: no longer U5.39 (GPIO27_ADC1)
- net GPIO28_ADC2: no longer U5.40 (GPIO28_ADC2)
- net GPIO29_ADC3: no longer U5.41 (GPIO29_ADC3)
- net GPIO3: no longer U5.5 (GPIO3)
- net QSPI_SCLK: no longer U5.52 (QSPI_SCLK), U6.6 (CLK)
- net QSPI_SD0: no longer U5.53 (QSPI_SD0), U6.5 (DI(IO0))
- net QSPI_SD1: no longer U5.55 (QSPI_SD1), U6.2 (DO(IO1))
- net QSPI_SD2: no longer U5.54 (QSPI_SD2), U6.3 (IO2)
- net QSPI_SD3: no longer U5.51 (QSPI_SD3), U6.7 (IO3)
- net QSPI_SS: no longer R18.1, R19.2, U5.56 (QSPI_SS), U6.1 (~{CS})
- net RUN: no longer U5.26 (RUN)
- net SWCLK: no longer U5.24 (SWCLK)
- net SWD: no longer U5.25 (SWD)
- net USB_D+: no longer J6.3 (D+), R20.1
- net USB_D-: no longer J6.2 (D-), R21.1
- net XIN: no longer C21.1, U5.20 (XIN), Y2.1
- net XOUT: no longer R17.1, U5.21 (XOUT)
- net ~{USB_BOOT}: no longer J7.1 (Pin_1), R18.2
- new net +3.3VP: C20.1, C27.1, C33.1, D38.2 (A), D39.2 (A), D40.2 (A), D41.2 (A), D42.2 (A), R19.1, U4.2 (VO), U6.8 (VCC)
- new net QSPI2_SCLK: U5.52 (QSPI_SCLK), U6.6 (CLK)
- new net QSPI2_SD0: U5.53 (QSPI_SD0), U6.5 (DI(IO0))
- new net QSPI2_SD1: U5.55 (QSPI_SD1), U6.2 (DO(IO1))
- new net QSPI2_SD2: U5.54 (QSPI_SD2), U6.3 (IO2)
- new net QSPI2_SD3: U5.51 (QSPI_SD3), U6.7 (IO3)
- new net QSPI2_SS: R18.1, R19.2, U5.56 (QSPI_SS), U6.1 (~{CS})
- new net USB2_D+: J6.3 (D+), R20.1
- new net USB2_D-: J6.2 (D-), R21.1
- new net XIN2: C21.1, U5.20 (XIN), Y2.1
- new net XOUT2: R17.1, U5.21 (XOUT)
- new net ~{USB2_BOOT}: J7.1 (Pin_1), R18.2

Commit message: ESD didoes to usb data lines added, fixed board 2 5V net name
Parts:
- added D47, D48, D49, D50: ESD5Zxx, Diode_SMD:D_SOD-523, symbol Diode:ESD5Zxx
Connections:
- net GND: now also D47.2 (A), D48.2 (A), D49.2 (A), D50.2 (A)
- net USB2_D+: now also D47.1 (K)
- net USB2_D-: now also D48.1 (K)
- net USB_D+: now also D50.1 (K)
- net USB_D-: now also D49.1 (K)
- net VBUS: no longer C23.1, J6.1 (VBUS), J8.1 (Pin_1), U4.3 (VI)
- new net +5VP: C23.1, J6.1 (VBUS), J8.1 (Pin_1), U4.3 (VI)

Commit message: added i2c breakout, and magnetic sensor to board 2
Parts:
- added C17, C37, C38, C39, C40, C41: DNP, Capacitor_SMD:C_0402_1005Metric, symbol Device:C
- added C42: 100n, Capacitor_SMD:C_0402_1005Metric, symbol Device:C
- added D51, D52: ESD5Zxx, Diode_SMD:D_SOD-523, symbol Diode:ESD5Zxx
- added J3: Conn_01x04, symbol Connector_Generic:Conn_01x04
- added R24, R25, R26, R27, R28, R29: 0, Capacitor_SMD:C_0402_1005Metric, symbol Device:R
- added R30: 10k, Capacitor_SMD:C_0402_1005Metric, symbol Device:R
- added U7: AH1806-W, Package_TO_SOT_SMD:SC-59, symbol Sensor_Magnetic:AH1806-W
Connections:
- net +3V3: now also C42.1, J3.1 (Pin_1), R30.2, U7.1 (VDD)
- net EN_SIG_A: now also U5.9 (GPIO7); no longer U5.3 (GPIO1)
- net EN_SIG_B: now also U5.8 (GPIO6); no longer U5.2 (GPIO0)
- net GND: now also C17.2, C37.2, C38.2, C39.2, C40.2, C41.2, C42.2, D51.2 (A), D52.2 (A), J3.4 (Pin_4), U7.3 (GND)
- net GPIO6: no longer U5.8 (GPIO6)
- net GPIO7: no longer U5.9 (GPIO7)
- net ROW0: now also C41.1, R24.2; no longer D1.1 (K), D2.1 (K), D3.1 (K), D4.1 (K), D5.1 (K), D6.1 (K), D7.1 (K)
- net ROW1: now also C40.1, R25.2; no longer D10.1 (K), D11.1 (K), D12.1 (K), D13.1 (K), D14.1 (K), D8.1 (K), D9.1 (K)
- net ROW2: now also C39.1, R26.2; no longer D15.1 (K), D16.1 (K), D17.1 (K), D18.1 (K), D19.1 (K), D20.1 (K)
- net ROW3: now also C38.1, R27.2; no longer D21.1 (K), D22.1 (K), D23.1 (K), D24.1 (K), D25.1 (K), D26.1 (K)
- net ROW4: now also C37.1, R28.2; no longer D27.1 (K), D28.1 (K), D29.1 (K), D30.1 (K), D31.1 (K), D32.1 (K)
- net ROW5: now also C17.1, R29.2; no longer D33.1 (K), D34.1 (K), D35.1 (K), D36.1 (K), D37.1 (K)
- net ~{Mag_Sensor}: now reaches U5.4 (GPIO2)
- net ~{Mag_Sensor}: now also R30.1, U7.2 (OUTPUT)
- new net: D1.1 (K), D2.1 (K), D3.1 (K), D4.1 (K), D5.1 (K), D6.1 (K), D7.1 (K), R24.1
- new net: D27.1 (K), D28.1 (K), D29.1 (K), D30.1 (K), D31.1 (K), D32.1 (K), R28.1
- new net: D21.1 (K), D22.1 (K), D23.1 (K), D24.1 (K), D25.1 (K), D26.1 (K), R27.1
- new net: D10.1 (K), D11.1 (K), D12.1 (K), D13.1 (K), D14.1 (K), D8.1 (K), D9.1 (K), R25.1
- new net: D33.1 (K), D34.1 (K), D35.1 (K), D36.1 (K), D37.1 (K), R29.1
- new net: D15.1 (K), D16.1 (K), D17.1 (K), D18.1 (K), D19.1 (K), D20.1 (K), R26.1
- new net I2C0_SCL: D52.1 (K), J3.2 (Pin_2), U5.3 (GPIO1)
- new net I2C0_SDA: D51.1 (K), J3.3 (Pin_3), U5.2 (GPIO0)
Other:
- note added: "Encoder_LEDs"
- note added: "I2C_Pin_Breakout"
- note added: "Magnetic Sensor"
- note added: "Rotary Encoder"
- moved on the sheet: C18, C19, C20, D1, D10, D11, D12, D13, D14, D15, D16, D17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

Commit message: forgot to add i2c to board 1
Parts:
- added D53, D54: ESD5Zxx, Diode_SMD:D_SOD-523, symbol Diode:ESD5Zxx
- added J4: Conn_01x04, symbol Connector_Generic:Conn_01x04
Connections:
- net +3V3: now also J4.1 (Pin_1)
- net GND: now also D53.2 (A), D54.2 (A), J4.4 (Pin_4)
- net I2C0_SCL: now also U3.3 (GPIO1), D54.1 (K), J4.2 (Pin_2); no longer D52.1 (K), J3.2 (Pin_2), U5.3 (GPIO1)
- net I2C0_SDA: now also U3.2 (GPIO0), D53.1 (K), J4.3 (Pin_3); no longer D51.1 (K), J3.3 (Pin_3), U5.2 (GPIO0)
- new net I2C0_SCL_2: D52.1 (K), J3.2 (Pin_2), U5.3 (GPIO1)
- new net I2C0_SDA_2: D51.1 (K), J3.3 (Pin_3), U5.2 (GPIO0)
